Commit message: realistic fridge model

File: models/simple_fridge.urdf (robot description, URDF)
Before this commit: robot myrobot, 3 links, 2 joints
Links:
- link base_link: geometry collision box size=0.57 0.53 1.5; visual box size=0.57 0.53 1.5
- link door_link: geometry collision box size=0.03 0.53 0.67; visual box size=0.03 0.53 0.67
- link handle_link: geometry visual box size=0.05 0.02 0.2
Joints:
- joint door_joint: origin xyz=-0.4 -0.4 0.85 rpy=0 0 0 -> xyz=-0.285 -0.265 0.83 rpy=0 0 0
- joint handle_joint: origin xyz=-0.03 0.72 0.17 rpy=0 0 0 -> xyz=-0.03 0.49 0.25 rpy=0 0 0

Commit message: completed demo

File: models/simple_fridge.urdf (robot description, URDF)
Before this commit: robot myrobot, 3 links, 2 joints
Links:
- link base_link: geometry collision box size=0.57 2.0 1.5; visual box size=0.57 0.53 1.5

Commit message: add desk

File: models/simple_fridge.urdf (robot description, URDF)
Before this commit: robot myrobot, 3 links, 2 joints
Links:
- added link desk_link; collision box size=0.8 1.2 0.7; visual box size=0.8 1.2 0.7
Joints:
- added joint desk_joint: type fixed, parent base_link, child desk_link, origin xyz=-2.3 0.8 0.0 rpy=0 0 0, axis 0 0 1

Commit message: add obstacle

File: models/simple_fridge.urdf (robot description, URDF)
Before this commit: robot myrobot, 4 links, 3 joints
Links:
- added link obstacle_link; collision box size=0.5 2.0 1.7; visual box size=0.5 2.0 1.7
- link base_link: geometry collision box size=0.57 0.53 1.5; visual box size=0.57 0.53 1.5
- link desk_link: geometry collision box size=0.8 1.2 0.1; visual box size=0.8 1.2 0.1
Joints:
- added joint obstacle_joint: type fixed, parent base_link, child obstacle_link, origin xyz=-0.15 1.4 0.0 rpy=0 0 0, axis 0 0 1

Commit message: Fix fridge location

File: models/simple_fridge.urdf (robot description, URDF)
Before this commit: robot myrobot, 5 links, 4 joints
Joints:
- joint desk_joint: origin xyz=-2.3 0.8 0.0 rpy=0 0 0 -> xyz=-2.1 0.8 0.0 rpy=0 0 0
