Commit message: Fix urdf structure

File: models/complecated_fridge.urdf (robot description, URDF)
Before this commit: robot myrobot, 9 links, 8 joints
Joints:
- joint base_back_joint: child base_link_top -> base_link_back

Commit message: Update model

File: models/complecated_fridge.urdf (robot description, URDF)
Before this commit: robot myrobot, 9 links, 8 joints
Links:
- added link base_link_middle; collision box size=0.57 0.53 0.85; visual box size=0.57 0.53 0.85
Joints:
- added joint base_middle_joint: type fixed, parent base_link, child base_link_middle, origin xyz=0.0 0.0 0.0 rpy=0 0 0, axis 0 0 1

Commit message: update fridge

File: models/complecated_fridge.urdf (robot description, URDF)
Before this commit: robot myrobot, 10 links, 9 joints
Links:
- removed link base_link_middle
- added link base_shelf_link; collision box size=0.4 0.53 0.3; visual box size=0.4 0.53 0.3
- link base_link: geometry collision box size=0.57 0.53 0.9; visual box size=0.57 0.53 0.9
Joints:
- removed joint base_middle_joint
- added joint base_shelf_joint: type fixed, parent base_link, child base_shelf_link, origin xyz=0.0 0.0 0.0 rpy=0 0 0, axis 0 0 1

Commit message: modify fridge shape

File: models/complecated_fridge.urdf (robot description, URDF)
Before this commit: robot myrobot, 10 links, 9 joints
Links:
- link base_link: geometry collision box size=0.57 0.53 0.99; visual box size=0.57 0.53 0.99

Commit message: add another obstacle

File: models/complecated_fridge.urdf (robot description, URDF)
Before this commit: robot myrobot, 10 links, 9 joints
Links:
- added link obstacle_link2; collision box size=1.5 1.0 1.7; visual box size=1.5 1.0 1.7
Joints:
- added joint obstacle_joint2: type fixed, parent base_link, child obstacle_link2, origin xyz=-0.8 1.6 0.0 rpy=0 0 0, axis 0 0 1

Commit message: update fridge model (thicker door)

File: models/complecated_fridge.urdf (robot description, URDF)
Before this commit: robot myrobot, 11 links, 10 joints
Links:
- link door_link: geometry collision box size=0.11 0.53 0.67; visual box size=0.11 0.53 0.67
Joints:
- joint door_joint: origin xyz=-0.285 -0.265 0.83 rpy=0 0 0 -> xyz=-0.23 -0.265 0.83 rpy=0 0 0
- joint handle_joint: origin xyz=-0.03 0.49 0.25 rpy=0 0 0 -> xyz=-0.06 0.49 0.25 rpy=0 0 0

Commit message: open lab stable version

File: models/complecated_fridge.urdf (robot description, URDF)
Before this commit: robot myrobot, 11 links, 10 joints
Links:
- removed link desk_link
Joints:
- removed joint desk_joint
